Commit message: Fixed transformation

File: description/manipulator.control.xacro (robot description, xacro)
@@ -1,77 +1,4 @@
 <?xml version="1.0" encoding="utf-8"?>
 <robot xmlns:xacro="http://www.ros.org/wiki/xacro" name="motoman_sia5f">
-    <gazebo>
-        <plugin filename="libgazebo_ros2_control.so" name="gazebo_ros2_control">
-            <parameters>$(find gazebo_simulation)/config/controllers.yaml</parameters>
-        </plugin>
-    </gazebo>
-    <ros2_control name="GazeboSystem" type="system">
-        <hardware>
-            <plugin>gazebo_ros2_control/GazeboSystem</plugin>
-            <robotSimType>gazebo_ros2_control/DefaultRobotHWSim</robotSimType>
-        </hardware>
-        <joint name="joint_s">
-            <command_interface name="position">
-                <!-- <param name="min">-2.8973</param> -->
-                <!-- <param name="max">2.8973</param> -->
-            </command_interface>
-            <state_interface name="position" />
-            <state_interface name="velocity" />
-            <state_interface name="effort" />
-        </joint>
-        <joint name="joint_l">
-            <command_interface name="position">
-                <!-- <param name="min">-1.7628</param> -->
-                <!-- <param name="max">1.7628</param> -->
-            </command_interface>
-            <state_interface name="position" />
-            <state_interface name="velocity" />
-            <state_interface name="effort" />
-        </joint>
-        <joint name="joint_e">
-            <command_interface name="position">
-                <!-- <param name="min">-2.8973</param> -->
-                <!-- <param name="max">2.8973</param> -->
-            </command_interface>
-            <state_interface name="position" />
-            <state_interface name="velocity" />
-            <state_interface name="effort" />
-        </joint>
-        <joint name="joint_u">
-            <command_interface name="position">
-                <!-- <param name="min">-3.0718</param> -->
-                <!-- <param name="max">-0.0698</param> -->
-            </command_interface>
-            <state_interface name="position" />
-            <state_interface name="velocity" />
-            <state_interface name="effort" />
-        </joint>
-        <joint name="joint_r">
-            <command_interface name="position">
-                <!-- <param name="min">-2.8973</param> -->
-                <!-- <param name="max">2.8973</param> -->
-            </command_interface>
-            <state_interface name="position" />
-            <state_interface name="velocity" />
-            <state_interface name="effort" />
-        </joint>
-        <joint name="joint_b">
-            <command_interface name="position">
-                <!-- <param name="min">-0.0175</param> -->
-                <!-- <param name="max">3.7525</param> -->
-            </command_interface>
-            <state_interface name="position" />
-            <state_interface name="velocity" />
-            <state_interface name="effort" />
-        </joint>
-        <joint name="joint_t">
-            <command_interface name="position">
-                <!-- <param name="min">-0.0175</param> -->
-                <!-- <param name="max">3.7525</param> -->
-            </command_interface>
-            <state_interface name="position" />
-            <state_interface name="velocity" />
-            <state_interface name="effort" />
-        </joint>
-    </ros2_control>
+    <xacro:include filename="$(find yaskawa_description)/robots/sia5f.control.xacro"/>
 </robot>

File: description/manipulator.gazebo.xacro (robot description, xacro)
@@ -1,104 +1,4 @@
 <?xml version="1.0" encoding="utf-8"?>
 <robot xmlns:xacro="http://www.ros.org/wiki/xacro" name="motoman_sia5f">
-    <!-- publishing the joint states to the /JointState topic-->
-    <gazebo>
-        <plugin name="gazebo_ros_joint_state_publisher" filename="libgazebo_ros_joint_state_publisher.so">
-            <update_rate>1000</update_rate>
-            <joint_name>joint_s</joint_name>
-            <joint_name>joint_l</joint_name>
-            <joint_name>joint_e</joint_name>
-            <joint_name>joint_u</joint_name>
-            <joint_name>joint_r</joint_name>
-            <joint_name>joint_b</joint_name>
-            <joint_name>joint_t</joint_name>
-        </plugin>
-    </gazebo>
-    <xacro:property name="robot_name" value="motoman_sia5f" />
-    <!-- Friction parameters-->
-    <gazebo reference="base_link">
-        <turnGravityOff>false</turnGravityOff>
-        <selfCollide>true</selfCollide>
-        <kp>0.0</kp>
-        <kd>0.0</kd>
-        <min_depth>0</min_depth>
-        <!-- <max_vel>0</max_vel> -->
-        <slip1>0</slip1>
-        <slip2>0</slip2>
-        <mu1>0</mu1>
-        <mu2>0</mu2>
-    </gazebo>
-    <!-- Link1 -->
-    <gazebo reference="link_s">
-        <turnGravityOff>false</turnGravityOff>
-        <selfCollide>true</selfCollide>
-        <material>Gazebo/White</material>
-        <kp>0.0</kp>
-        <kd>0.0</kd>
-        <min_depth>0</min_depth>
-        <!-- <max_vel>0</max_vel> -->
-        <slip1>0</slip1>
-        <slip2>0</slip2>
-        <mu1>0</mu1>
-        <mu2>0</mu2>
-    </gazebo>
-    <!-- Link2 -->
-    <gazebo reference="link_l">
-        <turnGravityOff>false</turnGravityOff>
-        <selfCollide>true</selfCollide>
-        <material>Gazebo/Blue</material>
-        <mu1>0.61</mu1>
-        <mu2>0.61</mu2>
-    </gazebo>
-    <!-- Link3 -->
-    <gazebo reference="link_e">
-        <turnGravityOff>false</turnGravityOff>
-        <selfCollide>true</selfCollide>
-        <material>Gazebo/White</material>
-        <mu1>0.61</mu1>
-        <mu2>0.61</mu2>
-    </gazebo>
-    <!-- Link4 -->
-    <gazebo reference="link_u">
-        <turnGravityOff>false</turnGravityOff>
-        <selfCollide>true</selfCollide>
-        <material>Gazebo/Blue</material>
-        <mu1>0.61</mu1>
-        <mu2>0.61</mu2>
-    </gazebo>
-    <!-- Link5 -->
-    <gazebo reference="link_r">
-        <turnGravityOff>false</turnGravityOff>
-        <selfCollide>true</selfCollide>
-        <material>Gazebo/White</material>
-        <mu1>0.61</mu1>
-        <mu2>0.61</mu2>
-    </gazebo>
-    <!-- Link6 -->
-    <gazebo reference="link_b">
-        <turnGravityOff>false</turnGravityOff>
-        <selfCollide>true</selfCollide>
-        <material>Gazebo/Blue</material>
-        <kp>100000.0</kp>
-        <kd>100.0</kd>
-        <min_depth>0</min_depth>
-        <!-- <max_vel>0</max_vel> -->
-        <slip1>0.2</slip1>
-        <slip2>0.2</slip2>
-        <mu>0.81</mu>
-        <mu2>0.5</mu2>
-    </gazebo>
-    <gazebo reference="link_t">
-        <turnGravityOff>false</turnGravityOff>
-        <selfCollide>true</selfCollide>
-        <material>Gazebo/White</material>
-        <!-- <kp>50000.0</kp> -->
-        <kp>50000.0</kp>
-        <kd>1.0</kd>
-        <min_depth>0</min_depth>
-        <!-- <max_vel>0</max_vel> -->
-        <slip1>0</slip1>
-        <slip2>0</slip2>
-        <mu1>0</mu1>
-        <mu2>0</mu2>
-    </gazebo>
+    <xacro:include filename="$(find yaskawa_description)/robots/sia5f.gazebo.xacro"/>
 </robot>

File: description/manipulator.urdf.xacro (robot description, xacro)
@@ -4,7 +4,10 @@
   <!-- <xacro:include filename="$(find yaskawa_description)/robots/sia5f_gazebo.xacro" />
   <xacro:sia5f_arm/>-->
-  <xacro:include filename="$(find gazebo_simulation)/description/yaskawa_wsg.xacro" />
+  <xacro:include filename="$(find gazebo_simulation)/description/yaskawa_pushing.xacro" />
   <xacro:manipulator/>
+  <xacro:include filename="$(find gazebo_simulation)/description/manipulator.control.xacro" />
   <xacro:include filename="$(find gazebo_simulation)/description/manipulator.gazebo.xacro" />
-  <xacro:include filename="$(find gazebo_simulation)/description/manipulator.control.xacro" />
+  <xacro:include filename="$(find gazebo_simulation)/description/camera.gazebo.xacro" />
+  <xacro:gazebo_d435 camera_name="camera_bottom" reference_link="camera_bottom_link" topics_ns="camera_bottom" depth_optical_frame="camera_bottom_depth_optical_frame" color_optical_frame="camera_bottom_color_optical_frame" infrared1_optical_frame="camera_bottom_infra1_optical_frame" infrared2_optical_frame="camera_bottom_infra2_optical_frame"></xacro:gazebo_d435>
+  <xacro:gazebo_d435 camera_name="camera_upper" reference_link="camera_upper_link" topics_ns="camera_upper" depth_optical_frame="camera_upper_depth_optical_frame" color_optical_frame="camera_upper_color_optical_frame" infrared1_optical_frame="camera_upper_infra1_optical_frame" infrared2_optical_frame="camera_upper_infra2_optical_frame"></xacro:gazebo_d435>
 </robot>

File: description/yaskawa_wsg.xacro (robot description, xacro)
@@ -5,5 +5,5 @@
         <xacro:include filename="$(find yaskawa_description)/robots/sia5f_arm.urdf"/>
         <xacro:include filename="$(find wsg32_description)/grippers/wsg32.urdf"/>
-        <xacro:wsg32_link base_link='base_link_gripper' xyz="-0.0002 -0.0076 -0.0007" rpy="0 3.14 -1.57" materials_="1"/>
+        <xacro:wsg32_link base_link='base_link_gripper' materials_="1"/>
         <joint name="tool0_joint_base_gripper" type="fixed">
             <origin xyz="0 0 0" rpy="${-90*deg} 0 ${-90*deg}"/>

Commit message: Fixed name

File: description/manipulator.control.xacro (robot description, xacro)
@@ -1,4 +1,4 @@
 <?xml version="1.0" encoding="utf-8"?>
 <robot xmlns:xacro="http://www.ros.org/wiki/xacro" name="motoman_sia5f">
-    <xacro:include filename="$(find yaskawa_description)/robots/sia5f.control.xacro"/>
+    <xacro:include filename="$(find yaskawa_description_ros2)/robots/sia5f.control.xacro"/>
 </robot>

File: description/manipulator.gazebo.xacro (robot description, xacro)
@@ -1,4 +1,4 @@
 <?xml version="1.0" encoding="utf-8"?>
 <robot xmlns:xacro="http://www.ros.org/wiki/xacro" name="motoman_sia5f">
-    <xacro:include filename="$(find yaskawa_description)/robots/sia5f.gazebo.xacro"/>
+    <xacro:include filename="$(find yaskawa_description_ros2)/robots/sia5f.gazebo.xacro"/>
 </robot>

File: description/manipulator.urdf.xacro (robot description, xacro)
@@ -2,5 +2,5 @@
 <robot xmlns:xacro="http://www.ros.org/wiki/xacro" name="motoman_sia5f">
   <xacro:property name="deg" value="0.017453293" />
-  <xacro:include filename="$(find gazebo_simulation)/description/yaskawa_pushing.xacro" />
+  <xacro:include filename="$(find gazebo_simulation_ros2)/description/yaskawa_pushing.xacro" />
   <xacro:manipulator/>
 </robot>

File: description/manipulator_all.urdf.xacro (robot description, xacro)
@@ -2,9 +2,9 @@
 <robot xmlns:xacro="http://www.ros.org/wiki/xacro" name="motoman_sia5f">
   <xacro:property name="deg" value="0.017453293" />
-  <xacro:include filename="$(find gazebo_simulation)/description/yaskawa_pushing.xacro" />
+  <xacro:include filename="$(find gazebo_simulation_ros2)/description/yaskawa_pushing.xacro" />
   <xacro:manipulator/>
-  <xacro:include filename="$(find gazebo_simulation)/description/manipulator.control.xacro" />
-  <xacro:include filename="$(find gazebo_simulation)/description/manipulator.gazebo.xacro" />
-  <xacro:include filename="$(find gazebo_simulation)/description/camera.gazebo.xacro" />
+  <xacro:include filename="$(find gazebo_simulation_ros2)/description/manipulator.control.xacro" />
+  <xacro:include filename="$(find gazebo_simulation_ros2)/description/manipulator.gazebo.xacro" />
+  <xacro:include filename="$(find gazebo_simulation_ros2)/description/camera.gazebo.xacro" />
   <xacro:gazebo_d435 camera_name="camera_bottom" reference_link="camera_bottom_link" topics_ns="camera_bottom" depth_optical_frame="camera_bottom_depth_optical_frame" color_optical_frame="camera_bottom_color_optical_frame" infrared1_optical_frame="camera_bottom_infra1_optical_frame" infrared2_optical_frame="camera_bottom_infra2_optical_frame"></xacro:gazebo_d435>
   <xacro:gazebo_d435 camera_name="camera_upper" reference_link="camera_upper_link" topics_ns="camera_upper" depth_optical_frame="camera_upper_depth_optical_frame" color_optical_frame="camera_upper_color_optical_frame" infrared1_optical_frame="camera_upper_infra1_optical_frame" infrared2_optical_frame="camera_upper_infra2_optical_frame"></xacro:gazebo_d435>

File: description/yaskawa_pushing.xacro (robot description, xacro)
@@ -4,6 +4,6 @@
         <xacro:property name="deg" value="0.017453293" />
         <!--degrees to radians-->
-        <xacro:include filename="$(find yaskawa_description)/robots/sia5f_arm.urdf"/>
-        <xacro:include filename="$(find gripper_description)/grippers/gripper_pushing.xacro"/>
+        <xacro:include filename="$(find yaskawa_description_ros2)/robots/sia5f_arm.urdf"/>
+        <xacro:include filename="$(find gripper_description_ros2)/grippers/gripper_pushing.xacro"/>
         <joint name="tool0_joint_base_gripper" type="fixed">
             <origin xyz="0 0 0" rpy="${-90*deg} 0 ${-90*deg}"/>

File: description/yaskawa_wsg.xacro (robot description, xacro)
@@ -3,6 +3,6 @@
     <xacro:macro name="manipulator">
         <xacro:property name="deg" value="0.017453293" /> <!--degrees to radians-->
-        <xacro:include filename="$(find yaskawa_description)/robots/sia5f_arm.urdf"/>
-        <xacro:include filename="$(find wsg32_description)/grippers/wsg32.urdf"/>
+        <xacro:include filename="$(find yaskawa_description_ros2)/robots/sia5f_arm.urdf"/>
+        <xacro:include filename="$(find wsg32_description_ros2)/grippers/wsg32.urdf"/>
         <xacro:wsg32_link base_link='base_link_gripper' materials_="1"/>
         <joint name="tool0_joint_base_gripper" type="fixed">
@@ -20,5 +20,5 @@
                 <origin xyz="0 0 0" rpy="0 0 0"/>
                 <geometry>
-                    <mesh filename="file://$(find gripper_description)/meshes/base_link.stl" scale="0.001 0.001 0.001"/>
+                    <mesh filename="file://$(find gripper_description_ros2)/meshes/base_link.stl" scale="0.001 0.001 0.001"/>
                 </geometry>
                 <material name="white1"/>
@@ -27,5 +27,5 @@
                 <origin xyz="0 0 0" rpy="0 0 0"/>
                 <geometry>
-                    <mesh filename="file://$(find gripper_description)/meshes/base_link.stl" scale="0.001 0.001 0.001"/>
+                    <mesh filename="file://$(find gripper_description_ros2)/meshes/base_link.stl" scale="0.001 0.001 0.001"/>
                 </geometry>
             </collision>
